File: loran_c_ethernet.sch (KiCad schematic (older format))
At the start: 39 parts, among them J201 RJ45, U201 LAN8720, X201 25MHz

Commit message: Update: fix, assign modules to components -Fix P302 incorrect connection -Assign footprints to components (not all yet) -Back-import footprints into schematic fields
Parts:
- C201, C203, C204, C208, C209, C210, C211: footprint (none) -> w_smd_capacitors:c_1206
- C202, C206: footprint (none) -> w_smd_capacitors:c_tant_A
- C205: footprint (none) -> w_smd_capacitors:c_0603
- C207: footprint (none) -> w_smd_capacitors:c_tant_B
- C212: footprint (none) -> w_pth_capacitors:cnp_6mm_disc
- D201: footprint (none) -> w_indicators:led_3mm_yellow
- D202: footprint (none) -> w_indicators:led_3mm_green
- FB201: footprint (none) -> w_pth_resistors:RC07
- MH201, MH202: footprint (none) -> Wire_Pads:SolderWirePad_single_2-5mmDrill
- R201, R202, R203, R204, R205, R206, R207, R208, R209, R210, R211, R212, R213, R214, R215, R216, R217, R218: footprint (none) -> w_smd_resistors:r_1206
- U201: footprint QFN24 -> w_smd_qfn:qfn-24
Other:
- note added: "RJ45 shield connects to\ndevice metal enclosure,\nNOT to digital ground!"
Changed lines of the file:
@@
 Date "18 янв. 2014"
 Rev ""
-Comp "Roman Dobrodiy"
+Comp "Roman Dobrodiy (aka RomaVis)"
 Comment1 ""
 Comment2 ""
@@
 F 0 "J201" H 9750 3550 60  0000 C CNN
 F 1 "RJ45" H 9400 3550 60  0000 C CNN
-F 2 "" H 9550 3050 60  0000 C CNN
+F 2 "" H 9550 3050 60  0001 C CNN
 F 3 "" H 9550 3050 60  0000 C CNN
 	1    9550 3050
@@
 F 0 "U201" H 5250 4450 50  0000 C CNN
 F 1 "LAN8720" H 4500 3400 50  0000 C CNN
-F 2 "QFN24" H 4500 3250 50  0000 C CNN
+F 2 "w_smd_qfn:qfn-24" H 4500 3250 50  0001 C CNN
 F 3 "" H 4200 3400 60  0001 C CNN
 	1    4500 3400
@@
 F 0 "TR201" H 7500 3450 50  0000 C CNN
 F 1 "TS8121" H 7500 2125 50  0000 C CNN
-F 2 "" H 7125 3150 60  0000 C CNN
+F 2 "" H 7125 3150 60  0001 C CNN
 F 3 "" H 7125 3150 60  0000 C CNN
 	1    7500 2850
@@
 F 0 "R208" V 6130 2050 40  0000 C CNN
 F 1 "49.9E 1%" V 6057 2051 40  0000 C CNN
-F 2 "" V 5980 2050 30  0000 C CNN
+F 2 "w_smd_resistors:r_1206" V 5980 2050 30  0001 C CNN
 F 3 "" H 6050 2050 30  0000 C CNN
 	1    6050 2050
@@
 F 0 "R210" V 6280 2050 40  0000 C CNN
 F 1 "49.9E 1%" V 6207 2051 40  0000 C CNN
-F 2 "" V 6130 2050 30  0000 C CNN
+F 2 "w_smd_resistors:r_1206" V 6130 2050 30  0001 C CNN
 F 3 "" H 6200 2050 30  0000 C CNN
 	1    6200 2050
@@
 F 0 "R212" V 6430 2050 40  0000 C CNN
 F 1 "49.9E 1%" V 6357 2051 40  0000 C CNN
-F 2 "" V 6280 2050 30  0000 C CNN
+F 2 "w_smd_resistors:r_1206" V 6280 2050 30  0001 C CNN
 F 3 "" H 6350 2050 30  0000 C CNN
 	1    6350 2050
@@
 F 0 "R213" V 6580 2050 40  0000 C CNN
 F 1 "49.9E 1%" V 6507 2051 40  0000 C CNN
-F 2 "" V 6430 2050 30  0000 C CNN
+F 2 "w_smd_resistors:r_1206" V 6430 2050 30  0001 C CNN
 F 3 "" H 6500 2050 30  0000 C CNN
 	1    6500 2050
@@
 F 0 "R215" V 8480 3850 40  0000 C CNN
 F 1 "75E 1%" V 8407 3851 40  0000 C CNN
-F 2 "" V 8330 3850 30  0000 C CNN
+F 2 "w_smd_resistors:r_1206" V 8330 3850 30  0001 C CNN
 F 3 "" H 8400 3850 30  0000 C CNN
 	1    8400 3850
@@
 F 0 "C212" H 9350 4250 40  0000 L CNN
 F 1 "1n 2000V" H 9356 4065 40  0000 L CNN
-F 2 "" H 9388 4000 30  0000 C CNN
+F 2 "w_pth_capacitors:cnp_6mm_disc" H 9388 4000 30  0001 C CNN
 F 3 "" H 9350 4150 60  0000 C CNN
 	1    9350 4150
@@
 F 0 "R216" V 8630 3850 40  0000 C CNN
 F 1 "75E 1%" V 8557 3851 40  0000 C CNN
-F 2 "" V 8480 3850 30  0000 C CNN
+F 2 "w_smd_resistors:r_1206" V 8480 3850 30  0001 C CNN
 F 3 "" H 8550 3850 30  0000 C CNN
 	1    8550 3850
@@
 F 0 "R217" V 8780 3850 40  0000 C CNN
 F 1 "75E 1%" V 8707 3851 40  0000 C CNN
-F 2 "" V 8630 3850 30  0000 C CNN
+F 2 "w_smd_resistors:r_1206" V 8630 3850 30  0001 C CNN
 F 3 "" H 8700 3850 30  0000 C CNN
 	1    8700 3850
@@
 F 0 "R218" V 8930 3850 40  0000 C CNN
 F 1 "75E 1%" V 8857 3851 40  0000 C CNN
-F 2 "" V 8780 3850 30  0000 C CNN
+F 2 "w_smd_resistors:r_1206" V 8780 3850 30  0001 C CNN
 F 3 "" H 8850 3850 30  0000 C CNN
 	1    8850 3850
@@
 F 0 "MH201" H 10550 3850 60  0000 C CNN
 F 1 "HOLE" H 10550 3470 60  0000 C CNN
-F 2 "" H 10550 3650 60  0000 C CNN
+F 2 "Wire_Pads:SolderWirePad_single_2-5mmDrill" H 10550 3650 60  0001 C CNN
 F 3 "" H 10550 3650 60  0000 C CNN
 	1    10550 3650
@@
 F 0 "MH202" H 10550 4350 60  0000 C CNN
 F 1 "HOLE" H 10550 3970 60  0000 C CNN
-F 2 "" H 10550 4150 60  0000 C CNN
+F 2 "Wire_Pads:SolderWirePad_single_2-5mmDrill" H 10550 4150 60  0001 C CNN
 F 3 "" H 10550 4150 60  0000 C CNN
 	1    10550 4150
@@
 F 0 "R207" V 4980 5250 40  0000 C CNN
 F 1 "12.1k 1%" V 4907 5251 40  0000 C CNN
-F 2 "" V 4830 5250 30  0000 C CNN
+F 2 "w_smd_resistors:r_1206" V 4830 5250 30  0001 C CNN
 F 3 "" H 4900 5250 30  0000 C CNN
 	1    4900 5250
@@
 F 0 "D201" H 6300 5150 50  0000 C CNN
 F 1 "LINK_SPEED" H 6300 4900 50  0000 C CNN
-F 2 "" H 6300 5050 60  0000 C CNN
+F 2 "w_indicators:led_3mm_yellow" H 6300 5050 60  0001 C CNN
 F 3 "" H 6300 5050 60  0000 C CNN
 	1    6300 5050
@@
 F 0 "R211" V 6380 4550 40  0000 C CNN
 F 1 "240" V 6307 4551 40  0000 C CNN
-F 2 "" V 6230 4550 30  0000 C CNN
+F 2 "w_smd_resistors:r_1206" V 6230 4550 30  0001 C CNN
 F 3 "" H 6300 4550 30  0000 C CNN
 	1    6300 4550
@@
 F 0 "R209" V 6130 4550 40  0000 C CNN
 F 1 "10k" V 6057 4551 40  0000 C CNN
-F 2 "" V 5980 4550 30  0000 C CNN
+F 2 "w_smd_resistors:r_1206" V 5980 4550 30  0001 C CNN
 F 3 "" H 6050 4550 30  0000 C CNN
 	1    6050 4550
@@
 F 0 "R214" V 6780 4550 40  0000 C CNN
 F 1 "240" V 6707 4551 40  0000 C CNN
-F 2 "" V 6630 4550 30  0000 C CNN
+F 2 "w_smd_resistors:r_1206" V 6630 4550 30  0001 C CNN
 F 3 "" H 6700 4550 30  0000 C CNN
 	1    6700 4550
@@
 F 0 "D202" H 6700 5150 50  0000 C CNN
 F 1 "LINK_ACT" H 6700 4900 50  0000 C CNN
-F 2 "" H 6700 5050 60  0000 C CNN
+F 2 "w_indicators:led_3mm_green" H 6700 5050 60  0001 C CNN
 F 3 "" H 6700 5050 60  0000 C CNN
 	1    6700 5050
@@
 F 0 "C206" H 4150 5350 50  0000 L CNN
 F 1 "2.2u 6.3V Ta" H 4100 5150 39  0000 L CNN
-F 2 "" H 4100 5250 60  0000 C CNN
+F 2 "w_smd_capacitors:c_tant_A" H 4100 5250 60  0001 C CNN
 F 3 "" H 4100 5250 60  0000 C CNN
 	1    4100 5250
@@
 F 0 "FB201" H 4100 1550 60  0000 C CNN
 F 1 "Bead" H 4100 1300 60  0000 C CNN
-F 2 "" H 4100 1400 60  0000 C CNN
+F 2 "w_pth_resistors:RC07" H 4100 1400 60  0001 C CNN
 F 3 "" H 4100 1400 60  0000 C CNN
 	1    4100 1400
@@
 F 0 "C209" H 7000 1750 40  0000 L CNN
 F 1 "10n" H 7006 1565 40  0000 L CNN
-F 2 "" H 7038 1500 30  0000 C CNN
+F 2 "w_smd_capacitors:c_1206" H 7038 1500 30  0001 C CNN
 F 3 "" H 7000 1650 60  0000 C CNN
 	1    7000 1650
@@
 F 0 "C210" H 7450 1750 40  0000 L CNN
 F 1 "10n" H 7456 1565 40  0000 L CNN
-F 2 "" H 7488 1500 30  0000 C CNN
+F 2 "w_smd_capacitors:c_1206" H 7488 1500 30  0001 C CNN
 F 3 "" H 7450 1650 60  0000 C CNN
 	1    7450 1650
@@
 F 0 "C207" H 5200 1750 50  0000 L CNN
 F 1 "10u 6.3V Ta" H 5200 1550 50  0000 L CNN
-F 2 "" H 5150 1650 60  0000 C CNN
+F 2 "w_smd_capacitors:c_tant_B" H 5150 1650 60  0001 C CNN
 F 3 "" H 5150 1650 60  0000 C CNN
 	1    5150 1650
@@
 F 0 "X201" H 2800 4800 60  0000 C CNN
 F 1 "25MHz" H 2800 4500 60  0000 C CNN
-F 2 "" H 2800 4650 60  0000 C CNN
+F 2 "" H 2800 4650 60  0001 C CNN
 F 3 "" H 2800 4650 60  0000 C CNN
 	1    2800 4650
@@
 F 0 "C203" H 3100 5250 40  0000 L CNN
 F 1 "22p" H 3106 5065 40  0000 L CNN
-F 2 "" H 3138 5000 30  0000 C CNN
+F 2 "w_smd_capacitors:c_1206" H 3138 5000 30  0001 C CNN
 F 3 "" H 3100 5150 60  0000 C CNN
 	1    3100 5150
@@
 F 0 "C201" H 2500 5250 40  0000 L CNN
 F 1 "22p" H 2506 5065 40  0000 L CNN
-F 2 "" H 2538 5000 30  0000 C CNN
+F 2 "w_smd_capacitors:c_1206" H 2538 5000 30  0001 C CNN
 F 3 "" H 2500 5150 60  0000 C CNN
 	1    2500 5150
@@
 F 0 "C211" H 7900 1750 40  0000 L CNN
 F 1 "22n" H 7906 1565 40  0000 L CNN
-F 2 "" H 7938 1500 30  0000 C CNN
+F 2 "w_smd_capacitors:c_1206" H 7938 1500 30  0001 C CNN
 F 3 "" H 7900 1650 60  0000 C CNN
 	1    7900 1650
@@
 F 0 "C205" H 3700 5350 40  0000 L CNN
 F 1 "470p" H 3706 5165 40  0000 L CNN
-F 2 "" H 3738 5100 30  0000 C CNN
+F 2 "w_smd_capacitors:c_0603" H 3738 5100 30  0001 C CNN
 F 3 "" H 3700 5250 60  0000 C CNN
 	1    3700 5250
@@
 F 0 "R205" V 2950 3850 40  0000 C CNN
 F 1 "33" V 2907 4051 40  0000 C CNN
-F 2 "" V 2830 4050 30  0000 C CNN
+F 2 "w_smd_resistors:r_1206" V 2830 4050 30  0001 C CNN
 F 3 "" H 2900 4050 30  0000 C CNN
 	1    2900 4050
@@
 F 0 "C208" H 5750 1750 40  0000 L CNN
 F 1 "100n" H 5756 1565 40  0000 L CNN
-F 2 "" H 5788 1500 30  0000 C CNN
+F 2 "w_smd_capacitors:c_1206" H 5788 1500 30  0001 C CNN
 F 3 "" H 5750 1650 60  0000 C CNN
 	1    5750 1650
@@
 F 0 "C202" H 2800 1750 50  0000 L CNN
 F 1 "2.2u 6.3V Ta" H 2800 1550 50  0000 L CNN
-F 2 "" H 2750 1650 60  0000 C CNN
+F 2 "w_smd_capacitors:c_tant_A" H 2750 1650 60  0001 C CNN
 F 3 "" H 2750 1650 60  0000 C CNN
 	1    2750 1650
@@
 F 0 "C204" H 3350 1750 40  0000 L CNN
 F 1 "100n" H 3356 1565 40  0000 L CNN
-F 2 "" H 3388 1500 30  0000 C CNN
+F 2 "w_smd_capacitors:c_1206" H 3388 1500 30  0001 C CNN
 F 3 "" H 3350 1650 60  0000 C CNN
 	1    3350 1650
@@
 F 0 "R206" V 2580 2450 40  0000 C CNN
 F 1 "1.5k" V 2507 2451 40  0000 C CNN
-F 2 "" V 2430 2450 30  0000 C CNN
+F 2 "w_smd_resistors:r_1206" V 2430 2450 30  0001 C CNN
 F 3 "" H 2500 2450 30  0000 C CNN
 	1    2500 2450
@@
 F 0 "R201" V 2950 2950 40  0000 C CNN
 F 1 "33" V 2907 3151 40  0000 C CNN
-F 2 "" V 2830 3150 30  0000 C CNN
+F 2 "w_smd_resistors:r_1206" V 2830 3150 30  0001 C CNN
 F 3 "" H 2900 3150 30  0000 C CNN
 	1    2900 3150
@@
 F 0 "R202" V 2950 3050 40  0000 C CNN
 F 1 "33" V 2907 3251 40  0000 C CNN
-F 2 "" V 2830 3250 30  0000 C CNN
+F 2 "w_smd_resistors:r_1206" V 2830 3250 30  0001 C CNN
 F 3 "" H 2900 3250 30  0000 C CNN
 	1    2900 3250
@@
 F 0 "R203" V 2950 3300 40  0000 C CNN
 F 1 "33" V 2907 3501 40  0000 C CNN
-F 2 "" V 2830 3500 30  0000 C CNN
+F 2 "w_smd_resistors:r_1206" V 2830 3500 30  0001 C CNN
 F 3 "" H 2900 3500 30  0000 C CNN
 	1    2900 3500
@@
 F 0 "R204" V 2950 3450 40  0000 C CNN
 F 1 "33" V 2907 3651 40  0000 C CNN
-F 2 "" V 2830 3650 30  0000 C CNN
+F 2 "w_smd_resistors:r_1206" V 2830 3650 30  0001 C CNN
 F 3 "" H 2900 3650 30  0000 C CNN
 	1    2900 3650
@@
 	1    0    0    -1
 $EndComp
+Text Notes 9950 4900 0    60   ~ 0
+RJ45 shield connects to\ndevice metal enclosure,\nNOT to digital ground!
 $EndSCHEMATC

Commit message: Intermediate update: PCB routing/schematic tweaking in process..
Parts:
- added C213, C214, C215, C216: 22n, w_smd_capacitors:c_1206, symbol C
Connections:
- net GND: now also C213.2, C214.2, C215.2, C216.2
- net RX+: now reaches J201.1, TR201.16 (TX+)
- net RX-: now reaches J201.2, TR201.14 (TX-)
- net TX+: now reaches J201.3, TR201.11 (RX+)
- net TX-: now reaches J201.6, TR201.9 (RX-)
- net PHY_VDDA: now reaches C207.1, C208.1, C209.1, C210.1, C211.1, FB201.2, R208.1, R210.1, R212.1, R213.1, TR201.2 (CT), TR201.7 (CT), U201.1 (VDD2A), U201.19 (VDD1A)
- net PHY_VDDA: now also C213.1, C214.1, C215.1, C216.1
- net LED2: now reaches R209.1, R211.1, U201.2 (LED2/nINTSEL)
- net RXN: now reaches R212.2, TR201.3 (TD-)
- net RXN: now also U201.22 (RXN); no longer U201.20 (TXN)
- net RXP: now reaches R213.2, TR201.1 (TD+)
- net RXP: now also U201.23 (RXP); no longer U201.21 (TXP)
- net TXN: now reaches R208.2, TR201.8 (RD-)
- net TXN: now also U201.20 (TXN); no longer U201.22 (RXN)
- net TXP: now reaches R210.2, TR201.6 (RD+)
- net TXP: now also U201.21 (TXP); no longer U201.23 (RXP)
- net LED1: now reaches R214.1, U201.3 (LED1/REGOFF)
- net XTAL2: now reaches C203.1, U201.4 (XTAL2), X201.2
- net XTAL1: now reaches C201.1, U201.5 (XTAL1/CLKIN), X201.1
- net VDDCR: now reaches C205.1, C206.1, U201.6 (VDDCR)
Other:
- note added: "Place caps close to:\nC211 - R212,R210\nC213 - pin 2 TR201\nC214 - pin 7 TR201\nC215 - R208\nC216 - R213"
- note added: "Swapping RX/TX enables better PCB routing\nDon't forget: AUTO-MDI/MDIX is supported"
- note removed: "Place close to\ntransformer pin 7!"

Commit message: Intermediate update #2: PCB routing/schematic tweaking in process
Parts:
- removed D201: LINK_SPEED, w_indicators:led_3mm_yellow, symbol LED
- removed D202: LINK_ACT, w_indicators:led_3mm_green, symbol LED
- removed MH201, MH202: HOLE, Wire_Pads:SolderWirePad_single_2-5mmDrill, symbol HOLE
- added C217: 100n, w_smd_capacitors:c_1206, symbol C
- added D201: LED_ETH, symbol LED_X2
- R206: value 1.5k -> 10k
Connections:
- wire segments 123 -> 125
Other:
- note added: "Place C204 close to pin 9 of U201"
- note added: "Swapping RX/TX of TR201 enables better PCB routing"
- note removed: "Swapping RX/TX enables better PCB routing\nDon't forget: AUTO-MDI/MDIX is supported"
- moved on the sheet: R211, R214
