File: loran_c_analog.sch (KiCad schematic (older format))
At the start: 62 parts, among them P601 DAC VCO, P602 DAC AGC, P603 QUAD In, P604 LORAN In, Q601 BD135, Q602 BD136, U601 TL072, U602 LD1117S33

Commit message: Update: PCB almost finished (3D views also up-to-date)
Parts:
- removed C616: 10u 6.3V Ta, w_smd_capacitors:c_tant_B, symbol CP1
- removed C623: 100n, w_smd_capacitors:c_1206, symbol C
- removed D603, D604: P6KE7V5 TVS, w_pth_diodes:diode_do15, symbol ZENER
- removed R609, R610, R616: Rt, w_pth_resistors:RC07, symbol R
- renumbered D605 to D603
Other:
- note removed: "Not fitted"
- moved on the sheet: C615, C617, C620, D603, P604, U602
