File: loran_c_relay.sch (KiCad schematic (older format))
At the start: 30 parts, among them IC501 PC817, IC502 PC817, P501 RELAY A, P502 RELAY B, P503 RELAY C, P504 RELAY D, Q401 BC847, Q402 BC847, Q403 BC847, Q501 BC847

Commit message: Update: PCB routing still in process...
Parts:
- removed C503: 2.2u 6.3V Ta, w_smd_capacitors:c_tant_B, symbol CP1
- renumbered Q401 to Q501, Q402 to Q502, Q403 to Q503, Q501 to Q504
Connections:
- net GND: now also P503.2 (PM), P504.2 (PM); no longer P503.1 (P1), P504.1 (P1)
- net at R505.2, R512.1: now also P503.1 (P1); no longer P503.2 (PM)
- net at R513.1, R514.2: now also P504.1 (P1); no longer P504.2 (PM)
- net RELAY1 renamed RELAY1_IN
- net RELAY2 renamed RELAY2_IN
- net RELAY3 renamed RELAY3_OUT
- net RELAY4 renamed RELAY4_OUT
Changed lines of the file:
@@
 LIBS:video
 LIBS:led_holder
+LIBS:crystal_shielded
 LIBS:loran_c_proc_board-cache
 EELAYER 24 0
@@
 $EndComp
 $Comp
-L GND #PWR098
+L GND #PWR096
 U 1 1 52DF2D2C
 P 5500 2400
-F 0 "#PWR098" H 5500 2400 30  0001 C CNN
+F 0 "#PWR096" H 5500 2400 30  0001 C CNN
 F 1 "GND" H 5500 2330 30  0001 C CNN
 F 2 "" H 5500 2400 60  0000 C CNN
@@
 $EndComp
 $Comp
-L GND #PWR099
+L GND #PWR097
 U 1 1 52DF2D32
 P 4400 2400
-F 0 "#PWR099" H 4400 2400 30  0001 C CNN
+F 0 "#PWR097" H 4400 2400 30  0001 C CNN
 F 1 "GND" H 4400 2330 30  0001 C CNN
 F 2 "" H 4400 2400 60  0000 C CNN
@@
 $EndComp
 $Comp
-L VDD #PWR0100
+L VDD #PWR098
 U 1 1 52DF2D44
 P 5150 1500
-F 0 "#PWR0100" H 5150 1600 30  0001 C CNN
+F 0 "#PWR098" H 5150 1600 30  0001 C CNN
 F 1 "VDD" H 5150 1610 30  0000 C CNN
 F 2 "" H 5150 1500 60  0000 C CNN
@@
 $EndComp
 $Comp
-L GND #PWR0101
+L GND #PWR099
 U 1 1 52DF2D68
 P 5500 3400
-F 0 "#PWR0101" H 5500 3400 30  0001 C CNN
+F 0 "#PWR099" H 5500 3400 30  0001 C CNN
 F 1 "GND" H 5500 3330 30  0001 C CNN
 F 2 "" H 5500 3400 60  0000 C CNN
@@
 $EndComp
 $Comp
-L GND #PWR0102
+L GND #PWR0100
 U 1 1 52DF2D6E
 P 4400 3400
-F 0 "#PWR0102" H 4400 3400 30  0001 C CNN
+F 0 "#PWR0100" H 4400 3400 30  0001 C CNN
 F 1 "GND" H 4400 3330 30  0001 C CNN
 F 2 "" H 4400 3400 60  0000 C CNN
@@
 F 3 "" H 7700 4450 60  0000 C CNN
 	1    7700 4450
-	1    0    0    1
+	1    0    0    -1
 $EndComp
 $Comp
@@
 F 3 "" H 7700 5500 60  0000 C CNN
 	1    7700 5500
-	1    0    0    1
+	1    0    0    -1
 $EndComp
 $Comp
@@
 $EndComp
 $Comp
-L GND #PWR0103
+L GND #PWR0101
 U 1 1 52DF2DFE
 P 5150 6250
-F 0 "#PWR0103" H 5150 6250 30  0001 C CNN
+F 0 "#PWR0101" H 5150 6250 30  0001 C CNN
 F 1 "GND" H 5150 6180 30  0001 C CNN
 F 2 "" H 5150 6250 60  0000 C CNN
@@
 $EndComp
 Text HLabel 3800 2150 0    60   Input ~ 0
-RELAY1
+RELAY1_IN
 Text HLabel 3800 3150 0    60   Input ~ 0
-RELAY2
+RELAY2_IN
 Text HLabel 3800 3900 0    60   Output ~ 0
-RELAY3
+RELAY3_OUT
 Text HLabel 3800 4950 0    60   Output ~ 0
-RELAY4
+RELAY4_OUT
 Text Notes 5650 1300 0    60   ~ 0
 Nominal optocoupler LED current: 10mA\n\nSchottky needed to protect optocoupler\ntransistors from reverse polarity voltage
 $Comp
-L BC849 Q401
+L BC849 Q501
 U 1 1 52E1A755
 P 5400 2150
-F 0 "Q401" H 5400 2001 40  0000 R CNN
+F 0 "Q501" H 5400 2001 40  0000 R CNN
 F 1 "BC847" H 5400 2300 40  0000 R CNN
 F 2 "SMD_Packages:SOT23" H 5300 2252 29  0001 C CNN
@@
 $EndComp
 $Comp
-L BC849 Q402
+L BC849 Q502
 U 1 1 52E1A773
 P 5400 3150
-F 0 "Q402" H 5400 3001 40  0000 R CNN
+F 0 "Q502" H 5400 3001 40  0000 R CNN
 F 1 "BC847" H 5400 3300 40  0000 R CNN
 F 2 "SMD_Packages:SOT23" H 5300 3252 29  0001 C CNN
@@
 $EndComp
 $Comp
-L BC849 Q403
+L BC849 Q503
 U 1 1 52E1A77E
 P 6100 4350
-F 0 "Q403" H 6100 4201 40  0000 R CNN
+F 0 "Q503" H 6100 4201 40  0000 R CNN
 F 1 "BC847" H 6100 4500 40  0000 R CNN
 F 2 "SMD_Packages:SOT23" H 6000 4452 29  0001 C CNN
@@
 $EndComp
 $Comp
-L GND #PWR0104
+L GND #PWR0102
 U 1 1 52F94D14
 P 7100 4600
-F 0 "#PWR0104" H 7100 4600 30  0001 C CNN
+F 0 "#PWR0102" H 7100 4600 30  0001 C CNN
 F 1 "GND" H 7100 4530 30  0001 C CNN
 F 2 "" H 7100 4600 60  0000 C CNN
@@
 $EndComp
 $Comp
-L GND #PWR0105
+L GND #PWR0103
 U 1 1 52F94FD4
 P 6000 4600
-F 0 "#PWR0105" H 6000 4600 30  0001 C CNN
+F 0 "#PWR0103" H 6000 4600 30  0001 C CNN
 F 1 "GND" H 6000 4530 30  0001 C CNN
 F 2 "" H 6000 4600 60  0000 C CNN
@@
 	7000 4350 7350 4350
 $Comp
-L GND #PWR0106
+L GND #PWR0104
 U 1 1 52F95259
 P 7300 4600
-F 0 "#PWR0106" H 7300 4600 30  0001 C CNN
+F 0 "#PWR0104" H 7300 4600 30  0001 C CNN
 F 1 "GND" H 7300 4530 30  0001 C CNN
 F 2 "" H 7300 4600 60  0000 C CNN
@@
 $EndComp
 $Comp
-L BC849 Q501
+L BC849 Q504
 U 1 1 52FABDCD
 P 6100 5400
-F 0 "Q501" H 6100 5251 40  0000 R CNN
+F 0 "Q504" H 6100 5251 40  0000 R CNN
 F 1 "BC847" H 6100 5550 40  0000 R CNN
 F 2 "SMD_Packages:SOT23" H 6000 5502 29  0001 C CNN
@@
 $EndComp
 $Comp
-L GND #PWR0107
+L GND #PWR0105
 U 1 1 52FABDD3
 P 7100 5650
-F 0 "#PWR0107" H 7100 5650 30  0001 C CNN
+F 0 "#PWR0105" H 7100 5650 30  0001 C CNN
 F 1 "GND" H 7100 5580 30  0001 C CNN
 F 2 "" H 7100 5650 60  0000 C CNN
@@
 $EndComp
 $Comp
-L GND #PWR0108
+L GND #PWR0106
 U 1 1 52FABDE5
 P 6000 5650
-F 0 "#PWR0108" H 6000 5650 30  0001 C CNN
+F 0 "#PWR0106" H 6000 5650 30  0001 C CNN
 F 1 "GND" H 6000 5580 30  0001 C CNN
 F 2 "" H 6000 5650 60  0000 C CNN
@@
 	7000 5400 7350 5400
 $Comp
-L GND #PWR0109
+L GND #PWR0107
 U 1 1 52FABDF3
 P 7300 5650
-F 0 "#PWR0109" H 7300 5650 30  0001 C CNN
+F 0 "#PWR0107" H 7300 5650 30  0001 C CNN
 F 1 "GND" H 7300 5580 30  0001 C CNN
 F 2 "" H 7300 5650 60  0000 C CNN
@@
 	1    0    0    -1
 $EndComp
-$Comp
-L CP1 C503
-U 1 1 52FAC7BB
-P 6700 6000
-F 0 "C503" H 6750 6100 50  0000 L CNN
-F 1 "2.2u 6.3V Ta" H 6750 5900 50  0000 L CNN
-F 2 "w_smd_capacitors:c_tant_B" H 6700 6000 60  0001 C CNN
-F 3 "" H 6700 6000 60  0000 C CNN
-	1    6700 6000
-	1    0    0    -1
-$EndComp
-Wire Wire Line
-	6700 5800 6700 5750
-Wire Wire Line
-	6700 5750 6350 5750
 Connection ~ 6350 5100
-Connection ~ 6350 5750
-$Comp
-L GND #PWR0110
+$Comp
+L GND #PWR0108
 U 1 1 52FAC89E
 P 6350 6250
-F 0 "#PWR0110" H 6350 6250 30  0001 C CNN
+F 0 "#PWR0108" H 6350 6250 30  0001 C CNN
 F 1 "GND" H 6350 6180 30  0001 C CNN
 F 2 "" H 6350 6250 60  0000 C CNN
@@
 	1    0    0    -1
 $EndComp
-$Comp
-L GND #PWR0111
-U 1 1 52FAC8A9
-P 6700 6250
-F 0 "#PWR0111" H 6700 6250 30  0001 C CNN
-F 1 "GND" H 6700 6180 30  0001 C CNN
-F 2 "" H 6700 6250 60  0000 C CNN
-F 3 "" H 6700 6250 60  0000 C CNN
-	1    6700 6250
-	1    0    0    -1
-$EndComp
-Wire Wire Line
-	6700 6200 6700 6250
 Wire Wire Line
 	6350 6200 6350 6250
