File: loran_c_rs232.sch (KiCad schematic (older format))
At the start: 27 parts, among them P301 UART1 3V3, P302 DB9 Ribbon 2, P303 DB9 Ribbon 1, U301 ST3232, U302 ST3232, U303 ST3232

Commit message: Update: PCB almost finished (3D views also up-to-date)
Parts:
- added P304: UART_SEL, symbol CONN_2S
Connections:
- net UART1_CTS: no longer U303.9 (R2OUT)
- net UART1_RX: no longer U303.12 (R1OUT)
- new net: P304.1 (P1), U303.12 (R1OUT)
- new net: P304.2 (PM), U303.9 (R2OUT)
Other:
- note added: "P304 pins 1 & 2 form jumper field with pins 2 & 3 of P301\n\nConnect pin 2(P301) with 1(P304), pin 3(P301) with 2(P304) to select RS232 UART1\nRemove these jumpers to use 3.3V UART1 (debug)"
- moved on the sheet: P301
Changed lines of the file:
@@
 LIBS:led_holder
 LIBS:crystal_shielded
+LIBS:conn_2s
 LIBS:loran_c_proc_board-cache
 EELAYER 24 0
@@
 DTE1_CTS
 $Comp
-L GND #PWR066
+L GND #PWR067
 U 1 1 52DBAE37
 P 5600 7750
-F 0 "#PWR066" H 5600 7750 30  0001 C CNN
+F 0 "#PWR067" H 5600 7750 30  0001 C CNN
 F 1 "GND" H 5600 7680 30  0001 C CNN
 F 2 "" H 5600 7750 60  0000 C CNN
@@
 DTE2_CTS
 $Comp
-L GND #PWR067
+L GND #PWR068
 U 1 1 52DBB093
 P 5600 3650
-F 0 "#PWR067" H 5600 3650 30  0001 C CNN
+F 0 "#PWR068" H 5600 3650 30  0001 C CNN
 F 1 "GND" H 5600 3580 30  0001 C CNN
 F 2 "" H 5600 3650 60  0000 C CNN
@@
 $EndComp
 $Comp
-L GND #PWR068
+L GND #PWR069
 U 1 1 52DBC5A6
 P 4900 2950
-F 0 "#PWR068" H 4900 2950 30  0001 C CNN
+F 0 "#PWR069" H 4900 2950 30  0001 C CNN
 F 1 "GND" H 4900 2880 30  0001 C CNN
 F 2 "" H 4900 2950 60  0000 C CNN
@@
 $EndComp
 $Comp
-L GND #PWR069
+L GND #PWR070
 U 1 1 52DBD4A5
 P 4900 7050
-F 0 "#PWR069" H 4900 7050 30  0001 C CNN
+F 0 "#PWR070" H 4900 7050 30  0001 C CNN
 F 1 "GND" H 4900 6980 30  0001 C CNN
 F 2 "" H 4900 7050 60  0000 C CNN
@@
 $EndComp
 $Comp
-L GND #PWR070
+L GND #PWR071
 U 1 1 52DBD9EF
 P 4900 5000
-F 0 "#PWR070" H 4900 5000 30  0001 C CNN
+F 0 "#PWR071" H 4900 5000 30  0001 C CNN
 F 1 "GND" H 4900 4930 30  0001 C CNN
 F 2 "" H 4900 5000 60  0000 C CNN
@@
 Text Label 1750 3400 0    61   ~ 0
 UART2_CTS
-Text Label 1750 7200 0    61   ~ 0
+Text Label 1350 7200 0    61   ~ 0
 UART1_TX
-Text Label 1750 7300 0    61   ~ 0
+Text Label 1350 7300 0    61   ~ 0
 UART1_RTS
-Text Label 1750 7400 0    61   ~ 0
+Text Label 1350 7400 0    61   ~ 0
 UART1_RX
-Text Label 1750 7500 0    61   ~ 0
+Text Label 1350 7500 0    61   ~ 0
 UART1_CTS
 $Comp
@@
 $EndComp
 $Comp
-L GND #PWR071
+L GND #PWR072
 U 1 1 52DC08D0
 P 5800 2500
-F 0 "#PWR071" H 5800 2500 30  0001 C CNN
+F 0 "#PWR072" H 5800 2500 30  0001 C CNN
 F 1 "GND" H 5800 2430 30  0001 C CNN
 F 2 "" H 5800 2500 60  0000 C CNN
@@
 $EndComp
 $Comp
-L GND #PWR072
+L GND #PWR073
 U 1 1 52DC08DB
 P 6150 2500
-F 0 "#PWR072" H 6150 2500 30  0001 C CNN
+F 0 "#PWR073" H 6150 2500 30  0001 C CNN
 F 1 "GND" H 6150 2430 30  0001 C CNN
 F 2 "" H 6150 2500 60  0000 C CNN
@@
 $EndComp
 $Comp
-L GND #PWR073
+L GND #PWR074
 U 1 1 52DC0F53
 P 7150 1650
-F 0 "#PWR073" H 7150 1650 30  0001 C CNN
+F 0 "#PWR074" H 7150 1650 30  0001 C CNN
 F 1 "GND" H 7150 1580 30  0001 C CNN
 F 2 "" H 7150 1650 60  0000 C CNN
@@
 $EndComp
 $Comp
-L VDD #PWR074
+L VDD #PWR075
 U 1 1 52DC1066
 P 7150 1050
-F 0 "#PWR074" H 7150 1150 30  0001 C CNN
+F 0 "#PWR075" H 7150 1150 30  0001 C CNN
 F 1 "VDD" H 7150 1160 30  0000 C CNN
 F 2 "" H 7150 1050 60  0000 C CNN
@@
 $EndComp
 $Comp
-L GND #PWR075
+L GND #PWR076
 U 1 1 52DC12C1
 P 5800 4550
-F 0 "#PWR075" H 5800 4550 30  0001 C CNN
+F 0 "#PWR076" H 5800 4550 30  0001 C CNN
 F 1 "GND" H 5800 4480 30  0001 C CNN
 F 2 "" H 5800 4550 60  0000 C CNN
@@
 $EndComp
 $Comp
-L GND #PWR076
+L GND #PWR077
 U 1 1 52DC12C7
 P 6150 4550
-F 0 "#PWR076" H 6150 4550 30  0001 C CNN
+F 0 "#PWR077" H 6150 4550 30  0001 C CNN
 F 1 "GND" H 6150 4480 30  0001 C CNN
 F 2 "" H 6150 4550 60  0000 C CNN
@@
 $EndComp
 $Comp
-L GND #PWR077
+L GND #PWR078
 U 1 1 52DC12FF
 P 5800 6600
-F 0 "#PWR077" H 5800 6600 30  0001 C CNN
+F 0 "#PWR078" H 5800 6600 30  0001 C CNN
 F 1 "GND" H 5800 6530 30  0001 C CNN
 F 2 "" H 5800 6600 60  0000 C CNN
@@
 $EndComp
 $Comp
-L GND #PWR078
+L GND #PWR079
 U 1 1 52DC1305
 P 6150 6600
-F 0 "#PWR078" H 6150 6600 30  0001 C CNN
+F 0 "#PWR079" H 6150 6600 30  0001 C CNN
 F 1 "GND" H 6150 6530 30  0001 C CNN
 F 2 "" H 6150 6600 60  0000 C CNN
@@
 L CONN_6 P301
 U 1 1 52DC1EFF
-P 1700 8300
-F 0 "P301" V 1650 8300 60  0000 C CNN
-F 1 "UART1 3V3" V 1750 8300 60  0000 C CNN
-F 2 "Pin_Headers:Pin_Header_Straight_1x06" H 1700 8300 60  0001 C CNN
-F 3 "" H 1700 8300 60  0000 C CNN
-	1    1700 8300
-	-1   0    0    -1
-$EndComp
-$Comp
-L GND #PWR079
-U 1 1 52DC2978
-P 2150 8650
-F 0 "#PWR079" H 2150 8650 30  0001 C CNN
-F 1 "GND" H 2150 8580 30  0001 C CNN
-F 2 "" H 2150 8650 60  0000 C CNN
-F 3 "" H 2150 8650 60  0000 C CNN
-	1    2150 8650
-	1    0    0    -1
-$EndComp
-Text Notes 2100 8050 0    61   ~ 0
+P 2500 8250
+F 0 "P301" V 2450 8250 60  0000 C CNN
+F 1 "UART1 3V3" V 2550 8250 60  0000 C CNN
+F 2 "Pin_Headers:Pin_Header_Straight_1x06" H 2500 8250 60  0001 C CNN
+F 3 "" H 2500 8250 60  0000 C CNN
+	1    2500 8250
+	1    0    0    -1
+$EndComp
+Text Notes 2050 8000 0    61   ~ 0
 Tx
-Text Notes 2100 8150 0    61   ~ 0
+Text Notes 2050 8100 0    61   ~ 0
 Rx
-Text Notes 2100 8350 0    61   ~ 0
+Text Notes 2000 8300 0    61   ~ 0
 RTS
-Text Notes 2100 8250 0    61   ~ 0
+Text Notes 2000 8200 0    61   ~ 0
 CTS
-Text Notes 2100 8450 0    61   ~ 0
+Text Notes 1700 8400 0    61   ~ 0
 DCD(PPS)
-Text Notes 2100 8550 0    61   ~ 0
+Text Notes 1950 8500 0    61   ~ 0
 GND
 NoConn ~ 6500 7350
@@
 	1200 7300 2750 7300
 Wire Wire Line
-	1200 7400 2750 7400
-Wire Wire Line
-	1200 7500 2750 7500
-Wire Wire Line
 	1200 5150 2750 5150
 Wire Wire Line
@@
 	4350 4050 6300 4050
 Wire Wire Line
-	2350 8050 2050 8050
-Wire Wire Line
-	2050 8150 2400 8150
-Wire Wire Line
-	2050 8250 2450 8250
-Wire Wire Line
-	2050 8350 2500 8350
-Wire Wire Line
-	2050 8450 2550 8450
-Wire Wire Line
-	2050 8550 2150 8550
-Wire Wire Line
-	2150 8550 2150 8650
-Wire Wire Line
 	6550 3450 6500 3450
 Wire Wire Line
@@
 Wire Wire Line
 	4350 5150 5550 5150
-Wire Wire Line
-	2350 8050 2350 7200
-Connection ~ 2350 7200
-Wire Wire Line
-	2400 8150 2400 7400
-Connection ~ 2400 7400
-Wire Wire Line
-	2450 8250 2450 7500
-Connection ~ 2450 7500
-Wire Wire Line
-	2500 8350 2500 7300
-Connection ~ 2500 7300
-Wire Wire Line
-	2550 8450 2550 7100
-Wire Wire Line
-	2550 7100 2250 7100
-Wire Wire Line
-	2250 7100 2250 5150
-Connection ~ 2250 5150
 $Comp
 L C C320
@@
 Wire Wire Line
 	5800 2050 5800 2000
+$Comp
+L CONN_2S P304
+U 1 1 5308B36A
+P 2700 8150
+F 0 "P304" V 2750 8150 40  0000 C CNN
+F 1 "UART_SEL" V 2650 8150 40  0000 C CNN
+F 2 "" H 2700 8150 60  0000 C CNN
+F 3 "" H 2700 8150 60  0000 C CNN
+	1    2700 8150
+	-1   0    0    -1
+$EndComp
+Text Notes 850  9150 0    63   ~ 0
+P304 pins 1 & 2 form jumper field with pins 2 & 3 of P301\n\nConnect pin 2(P301) with 1(P304), pin 3(P301) with 2(P304) to select RS232 UART1\nRemove these jumpers to use 3.3V UART1 (debug)
+Wire Wire Line
+	2150 8000 2000 8000
+Wire Wire Line
+	2000 8000 2000 7200
+Connection ~ 2000 7200
+Wire Wire Line
+	2150 8100 1950 8100
+Wire Wire Line
+	1950 8100 1950 7400
+Wire Wire Line
+	2150 8200 1900 8200
+Wire Wire Line
+	1900 8200 1900 7500
+Wire Wire Line
+	2150 8300 1850 8300
+Wire Wire Line
+	1850 8300 1850 7300
+Connection ~ 1850 7300
+Wire Wire Line
+	2150 8400 1300 8400
+Wire Wire Line
+	1300 8400 1300 5150
+Connection ~ 1300 5150
+Wire Wire Line
+	2150 8500 2050 8500
+Wire Wire Line
+	2050 8500 2050 8600
+$Comp
+L GND #PWR082
+U 1 1 5308BE15
+P 2050 8600
+F 0 "#PWR082" H 2050 8600 30  0001 C CNN
+F 1 "GND" H 2050 8530 30  0001 C CNN
+F 2 "" H 2050 8600 60  0000 C CNN
+F 3 "" H 2050 8600 60  0000 C CNN
+	1    2050 8600
+	1    0    0    -1
+$EndComp
+Wire Wire Line
+	1950 7400 1200 7400
+Wire Wire Line
+	1900 7500 1200 7500
+Wire Wire Line
+	3050 8100 3100 8100
+Wire Wire Line
+	3100 8100 3100 7850
+Wire Wire Line
+	3100 7850 2550 7850
+Wire Wire Line
+	2550 7850 2550 7400
+Wire Wire Line
+	2550 7400 2750 7400
+Wire Wire Line
+	3050 8200 3200 8200
+Wire Wire Line
+	3200 8200 3200 7750
+Wire Wire Line
+	3200 7750 2650 7750
+Wire Wire Line
+	2650 7750 2650 7500
+Wire Wire Line
+	2650 7500 2750 7500
 $EndSCHEMATC
