File: loran_c_proc_board.kicad_pcb (KiCad board)
At the start: 2 copper layers, 160 x 104.1 mm, 236 parts, among them IC501 PC817, IC502 PC817, IC503 PC817, IC504 PC817, J201 RJ45, P101 Power, P102 Cortex SWD, P103 Clock board, P301 UART1 3V3, P302 DB9 Ribbon 1, P303 DB9 Ribbon 2, P401 SPI Bus A, P402 SPI Bus B, P501 RELAY A, P502 RELAY B, P503 RELAY C, P504 RELAY D, P601 DAC VCO, P602 DAC AGC, P603 LORAN In, P604 RSVD In, Q401 BC847, Q402 BC847, Q403 BC847, Q404 BC847, Q601 BD135, Q602 BD136, U101 LD1117S33, U102 74AC14, U103 74AC14, U201 LAN8720, U301 ST3232, U302 ST3232, U303 ST3232, U401 74AC14, U402 74AC14, U601 TL072, U602 LD1117S33, U701 STM32F407VG, X201 25MHz, X701 32.768KHz

Commit message: Intermediate update: PCB routing/schematic tweaking in process..
Parts:
- removed C320, C321: 100n, w_smd_capacitors:c_1206
- removed FB302, FB303: Bead, w_pth_resistors:RC07
- added C213: 22n, w_smd_capacitors:c_1206, B.Cu at (197.2, 83.6)
- added C214: 22n, w_smd_capacitors:c_1206, B.Cu at (197.2, 89.9)
- added C215: 22n, w_smd_capacitors:c_1206, B.Cu at (190.4, 93.1)
- added C216: 22n, w_smd_capacitors:c_1206, B.Cu at (190.4, 80.4)
- added C405: 100n, w_smd_capacitors:c_1206, F.Cu at (122.4, 109.3)
- C201, C203: footprint w_smd_capacitors:c_1206 -> w_smd_resistors:r_0805; moved to B.Cu
- C204, C211, C314, C315, C316, C317, C318, C319, C601, C602, C609, C610, C611, C612, C708, C712, C713, D607, D609, R605, R606, R607, R608: moved to B.Cu
- C205: footprint w_smd_capacitors:c_0603 -> w_smd_resistors:r_0805
- R201, R202, R203, R204, R205: footprint w_smd_resistors:r_1206 -> w_smd_resistors:r_0805
- R609, R610: footprint w_pth_resistors:RC07 -> w_smd_resistors:r_1210
- moved R718 246.7 mm to (-19.9, 23.2)
- moved R717 246.0 mm to (-19.9, 20.8)
- moved R716 245.5 mm to (-19.9, 25.7)
- moved R702 243.4 mm to (19.5, 30.8)
- moved R705 243.4 mm to (19.5, 34.7)
- moved C701 243.4 mm to (30.3, 26.2)
- moved C702 243.4 mm to (-0.89, 40.3)
- moved C703 243.4 mm to (20.5, 22.8)
- moved C704 243.4 mm to (4.51, 28.2)
- moved C711 243.4 mm to (-6.08, 41.0)
- moved FB701 243.4 mm to (-7.37, 16.6)
- moved JP702 243.4 mm to (-12.1, 41.9)
- moved R701 243.4 mm to (8.91, 41.5)
- moved R707 243.4 mm to (30.3, 22.1)
- moved R708 243.4 mm to (14.0, 38.1)
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Connections:
- net Net-(C201-Pad1) renamed /Ethernet PHY/XTAL1
- net Net-(C203-Pad1) renamed /Ethernet PHY/XTAL2
- net Net-(C205-Pad1) renamed /Ethernet PHY/VDDCR
- net Net-(C207-Pad1) renamed /Ethernet PHY/PHY_VDDA
- net Net-(C603-Pad1) renamed /Analog part/+15V_AS
- net Net-(C604-Pad2) renamed /Analog part/-15V_AS
- net Net-(J201-Pad1) renamed /Ethernet PHY/RX+
- net Net-(J201-Pad2) renamed /Ethernet PHY/RX-
- net Net-(J201-Pad3) renamed /Ethernet PHY/TX+
- net Net-(J201-Pad6) renamed /Ethernet PHY/TX-
- net Net-(R209-Pad1) renamed /Ethernet PHY/LED2
- net Net-(R214-Pad1) renamed /Ethernet PHY/LED1
- C313 pad 1: Net-(C313-Pad1) -> /RS232 interface/RS232_PWR
- C314 pad 1: Net-(C314-Pad1) -> /RS232 interface/RS232_PWR
- C315 pad 1: Net-(C315-Pad1) -> /RS232 interface/RS232_PWR
- C316 pad 1: Net-(C313-Pad1) -> /RS232 interface/RS232_PWR
- C317 pad 1: Net-(C314-Pad1) -> /RS232 interface/RS232_PWR
- C318 pad 1: Net-(C315-Pad1) -> /RS232 interface/RS232_PWR
- FB301 pad 1: Net-(C313-Pad1) -> /RS232 interface/RS232_PWR
- P101 pad 3: /Analog part/+15V -> AGND
- P101 pad 4: AGND -> /Analog part/+15V
- R208 pad 2: Net-(R208-Pad2) -> /Ethernet PHY/TXN
- R210 pad 2: Net-(R210-Pad2) -> /Ethernet PHY/TXP
- R212 pad 2: Net-(R212-Pad2) -> /Ethernet PHY/RXN
- R213 pad 2: Net-(R213-Pad2) -> /Ethernet PHY/RXP
- TR201 pad 1: Net-(R213-Pad2) -> /Ethernet PHY/RXP
- TR201 pad 3: Net-(R212-Pad2) -> /Ethernet PHY/RXN
- TR201 pad 6: Net-(R210-Pad2) -> /Ethernet PHY/TXP
- TR201 pad 8: Net-(R208-Pad2) -> /Ethernet PHY/TXN
- U201 pad 20: Net-(R212-Pad2) -> /Ethernet PHY/TXN
- U201 pad 21: Net-(R213-Pad2) -> /Ethernet PHY/TXP
- U201 pad 22: Net-(R208-Pad2) -> /Ethernet PHY/RXN
- U201 pad 23: Net-(R210-Pad2) -> /Ethernet PHY/RXP
- U301 pad 16: Net-(C313-Pad1) -> /RS232 interface/RS232_PWR
- U302 pad 10: /uC STM32F407/PPS2 -> /uC STM32F407/PPS1
- U302 pad 11: /uC STM32F407/PPS1 -> /uC STM32F407/PPS2
- U302 pad 14: /RS232 interface/DTE1_DCD -> /RS232 interface/DTE2_DCD
- U302 pad 16: Net-(C314-Pad1) -> /RS232 interface/RS232_PWR
- U302 pad 7: /RS232 interface/DTE2_DCD -> /RS232 interface/DTE1_DCD
- U303 pad 16: Net-(C315-Pad1) -> /RS232 interface/RS232_PWR
- U601 pad 1: Net-(R605-Pad1) -> Net-(R606-Pad1)
- U601 pad 2: Net-(R605-Pad1) -> Net-(R606-Pad1)
- U601 pad 3: Net-(C601-Pad1) -> Net-(C602-Pad2)
- U601 pad 5: Net-(C602-Pad2) -> Net-(C601-Pad1)
- U601 pad 6: Net-(R606-Pad1) -> Net-(R605-Pad1)
- U601 pad 7: Net-(R606-Pad1) -> Net-(R605-Pad1)
Routing:
- net AGND: track 75.2 -> 216.0 mm, vias 0 -> 3
- net /RS232 interface/RS232_PWR: track 0.00 -> 93.7 mm, vias 0 -> 6
- net /Ethernet PHY/PHY_VDDA: track 0.00 -> 91.7 mm, vias 0 -> 14
- net +3.3VADC: track 0.00 -> 60.6 mm, vias 0 -> 14
- net VDD: track 47.3 -> 96.8 mm
- net -7.5V: track 43.0 -> 92.3 mm
- net +7.5V: track 43.1 -> 87.6 mm
- net /Analog part/-15V_AS: track 53.5 -> 92.4 mm
- net /uC STM32F407/ADC1_IN: track 0.00 -> 35.8 mm
- net Net-(R605-Pad1): track 0.00 -> 34.5 mm
- net /uC STM32F407/ADC2_IN: track 0.00 -> 31.9 mm
- net Net-(R606-Pad1): track 0.00 -> 31.6 mm
- net /RS232 interface/DTE2_DCD: track 0.00 -> 31.5 mm
- net /RS232 interface/DTE1_DCD: track 0.00 -> 26.6 mm
- net /Ethernet PHY/TXN: track 0.00 -> 23.4 mm
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- added copper zone on B.Cu, net +3.3VADC
- added copper zone on F.Cu, net +3.3VADC
- added copper zone on F.Cu, net /Analog part/+15V_AS
- added copper zone on F.Cu, net /Analog part/-15V_AS
- added copper zone on B.Cu, net /Ethernet PHY/PHY_VDDA
- added copper zone on F.Cu, net /Ethernet PHY/PHY_VDDA
- added copper zone on B.Cu, net GND
- added copper zone on F.Cu, net GND
Other:
- net class 3v3_power: clearance 0.254 -> 0.15
- net class Default: clearance 0.254 -> 0.15
- rule trace_clearance: 0.254 -> 0.15
- rule trace_min: 0.254 -> 0.15
- rule via_min_drill: 0.5 -> 0.2
- rule via_min_size: 1 -> 0.7

Commit message: Intermediate update #2: PCB routing/schematic tweaking in process
Parts:
- removed D202: LINK_ACT, w_indicators:led_3mm_green
- removed MH201, MH202: HOLE, Wire_Pads:SolderWirePad_single_2-5mmDrill
- removed R705, R714: 33, w_smd_resistors:r_1206
- added BT101: Li CR2032, w_battery_holders:keystone_103, F.Cu at (151.6, 156.9)
- added C217: 100n, w_smd_capacitors:c_1206, B.Cu at (188.8, 74.9)
- added C716: 100n, w_smd_capacitors:c_0805, B.Cu at (141.8, 78.5)
- added MH101: HOLE, holes:Hole_3-5mm, F.Cu at (64.5, 43.6)
- added MH102: HOLE, holes:Hole_3-5mm, F.Cu at (64.5, 123.6)
- added MH103: HOLE, holes:Hole_3-5mm, F.Cu at (209.5, 123.6)
- added MH104: HOLE, holes:Hole_3-5mm, F.Cu at (209.5, 43.6)
- added R719: 33, w_smd_resistors:r_1206, F.Cu at (157.3, 93.0)
- added R720: 1.5k, w_smd_resistors:r_0805, F.Cu at (139.5, 86.6)
- C207, C208, C714, C715, R704: moved to B.Cu
- C706, C707, C708, C709: footprint w_smd_capacitors:c_1206 -> w_smd_capacitors:c_0805
- C710: footprint w_smd_capacitors:c_1206 -> w_smd_capacitors:c_0805; moved to B.Cu
- C712, C713, R401: moved to F.Cu
- D201: value LINK_SPEED -> LED_ETH; footprint w_indicators:led_3mm_yellow -> led_holder:LED-306
- FB103: footprint w_pth_resistors:RC07 -> w_smd_resistors:r_0805; moved to B.Cu
- P302: value DB9 Ribbon 1 -> DB9 Ribbon 2
- P303: value DB9 Ribbon 2 -> DB9 Ribbon 1
- R201, R202: footprint w_smd_resistors:r_0805 -> w_smd_resistors:r_1206
- R206: value 1.5k -> 10k
- R709, R710: footprint w_smd_resistors:r_1206 -> w_smd_resistors:r_0805
- R715: footprint w_smd_resistors:r_1206 -> w_smd_resistors:r_0805; moved to B.Cu
- moved C702 264.2 mm to (223.6, 179.5)
- moved C703 264.2 mm to (245.0, 162.0)
- moved C704 264.2 mm to (229.0, 167.4)
- moved C705 264.2 mm to (234.9, 163.4)
- moved C711 264.2 mm to (218.4, 180.2)
- moved D702 264.2 mm to (228.9, 172.4)
- moved FB701 264.2 mm to (217.1, 155.8)
- moved R701 264.2 mm to (233.4, 180.7)
- moved R702 264.2 mm to (244.0, 170.0)
- moved R703 264.2 mm to (228.5, 180.7)
- moved R711 264.2 mm to (240.1, 165.4)
- moved R712 264.2 mm to (239.1, 173.3)
- moved R713 264.2 mm to (234.2, 172.1)
- moved R717 174.0 mm to (147.9, 66.9), turned to 180 degrees
- moved R718 170.6 mm to (144.4, 69.2), turned to 180 degrees
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Connections:
- J201 pad 1: /Ethernet PHY/RX+ -> /Ethernet PHY/TX+
- J201 pad 2: /Ethernet PHY/RX- -> /Ethernet PHY/TX-
- J201 pad 3: /Ethernet PHY/TX+ -> /Ethernet PHY/RX+
- J201 pad 6: /Ethernet PHY/TX- -> /Ethernet PHY/RX-
- P301 pad 3: /RS232 interface/UART1_RTS -> /RS232 interface/UART1_CTS
- P301 pad 4: /RS232 interface/UART1_CTS -> /RS232 interface/UART1_RTS
- P302 pad 1: /RS232 interface/DTE1_DCD -> /RS232 interface/DTE2_DCD
- P302 pad 2: /RS232 interface/DTE1_RxD -> /RS232 interface/DTE2_RxD
- P302 pad 3: /RS232 interface/DTE1_TxD -> /RS232 interface/DTE2_TxD
- P302 pad 7: /RS232 interface/DTE1_RTS -> /RS232 interface/DTE2_RTS
- P302 pad 8: /RS232 interface/DTE1_CTS -> /RS232 interface/DTE2_CTS
- P303 pad 1: /RS232 interface/DTE2_DCD -> /RS232 interface/DTE1_DCD
- P303 pad 2: /RS232 interface/DTE2_RxD -> /RS232 interface/DTE1_RxD
- P303 pad 3: /RS232 interface/DTE2_TxD -> /RS232 interface/DTE1_TxD
- P303 pad 7: /RS232 interface/DTE2_RTS -> /RS232 interface/DTE1_RTS
- P303 pad 8: /RS232 interface/DTE2_CTS -> /RS232 interface/DTE1_CTS
- R206 pad 1: /Ethernet PHY/RMII_MDIO -> /Ethernet PHY/LED1
- R206 pad 2: VDD -> GND
- R211 pad 2: Net-(D201-Pad1) -> Net-(D201-Pad3)
- R214 pad 2: Net-(D202-Pad1) -> Net-(D201-Pad1)
- R716 pad 1: Net-(R716-Pad1) -> /SPI interface/SPI_STRB
- R716 pad 2: /SPI interface/SPI_STRB -> Net-(R716-Pad2)
- R717 pad 1: Net-(R717-Pad1) -> /SPI interface/SPI_SCK
- R717 pad 2: /SPI interface/SPI_SCK -> Net-(R717-Pad2)
- R718 pad 1: Net-(R718-Pad1) -> /SPI interface/SPI_MOSI
- R718 pad 2: /SPI interface/SPI_MOSI -> Net-(R712-Pad1)
- U301 pad 10: /RS232 interface/UART1_RTS -> /RS232 interface/UART2_RTS
- U301 pad 11: /RS232 interface/UART1_TX -> /RS232 interface/UART2_TX
- U301 pad 12: /RS232 interface/UART1_RX -> /RS232 interface/UART2_RX
- U301 pad 13: /RS232 interface/DTE1_TxD -> /RS232 interface/DTE2_TxD
- U301 pad 14: /RS232 interface/DTE1_RxD -> /RS232 interface/DTE2_RxD
- U301 pad 7: /RS232 interface/DTE1_CTS -> /RS232 interface/DTE2_CTS
- U301 pad 8: /RS232 interface/DTE1_RTS -> /RS232 interface/DTE2_RTS
- U301 pad 9: /RS232 interface/UART1_CTS -> /RS232 interface/UART2_CTS
- U302 pad 10: /uC STM32F407/PPS1 -> /uC STM32F407/PPS2
- U302 pad 11: /uC STM32F407/PPS2 -> /uC STM32F407/PPS1
- U302 pad 14: /RS232 interface/DTE2_DCD -> /RS232 interface/DTE1_DCD
- U302 pad 7: /RS232 interface/DTE1_DCD -> /RS232 interface/DTE2_DCD
- U303 pad 10: /RS232 interface/UART2_RTS -> /RS232 interface/UART1_RTS
- U303 pad 11: /RS232 interface/UART2_TX -> /RS232 interface/UART1_TX
- U303 pad 12: /RS232 interface/UART2_RX -> /RS232 interface/UART1_RX
- U303 pad 13: /RS232 interface/DTE2_TxD -> /RS232 interface/DTE1_TxD
- U303 pad 14: /RS232 interface/DTE2_RxD -> /RS232 interface/DTE1_RxD
- U303 pad 7: /RS232 interface/DTE2_CTS -> /RS232 interface/DTE1_CTS
- U303 pad 8: /RS232 interface/DTE2_RTS -> /RS232 interface/DTE1_RTS
- U303 pad 9: /RS232 interface/UART2_CTS -> /RS232 interface/UART1_CTS
- U701 pad 16: Net-(R714-Pad1) -> /Ethernet PHY/RMII_MDC
- U701 pad 23: GND -> (no net)
- U701 pad 25: Net-(R705-Pad2) -> /Ethernet PHY/RMII_MDIO
- U701 pad 47: /Ethernet PHY/RMII_NRST -> Net-(R719-Pad2)
- U701 pad 78: Net-(R717-Pad1) -> (no net)
- U701 pad 79: /SPI interface/SPI_MISO -> (no net)
- U701 pad 80: Net-(R718-Pad1) -> (no net)
- U701 pad 81: Net-(R716-Pad1) -> (no net)
- U701 pad 89: (no net) -> Net-(R717-Pad2)
- U701 pad 90: (no net) -> /SPI interface/SPI_MISO
- U701 pad 92: (no net) -> Net-(R716-Pad2)
- X701 pad 1: /uC STM32F407/LSE_OUT -> /uC STM32F407/LSE_IN
- X701 pad 2: /uC STM32F407/LSE_IN -> /uC STM32F407/LSE_OUT
Routing:
- net VDD: track 96.8 -> 147.2 mm, vias 0 -> 6
- net /Relay optoisolation/RELAY1: track 0.00 -> 48.4 mm
- net /SPI interface/SPI_MISO: track 25.4 -> 72.5 mm
- net /Relay optoisolation/RELAY2: track 0.00 -> 40.2 mm
- net /SPI interface/SPI_SCK: track 48.2 -> 87.8 mm
- net /RS232 interface/UART2_RX: track 0.00 -> 38.6 mm
- net /SPI interface/SPI_MOSI: track 16.0 -> 53.6 mm
- net /uC STM32F407/PPS1: track 4.68 -> 42.2 mm, vias 0 -> 2
- net /Ethernet PHY/RMII_MDIO: track 0.00 -> 36.6 mm
- net /RS232 interface/UART2_TX: track 0.00 -> 36.5 mm
- net /RS232 interface/UART2_RTS: track 0.00 -> 34.8 mm
- net /uC STM32F407/PPS2: track 6.41 -> 40.8 mm, vias 0 -> 2
- net /SPI interface/SPI_STRB: track 51.0 -> 85.2 mm
- net /Analog part/-15V_AS: track 92.4 -> 59.4 mm
- net /RS232 interface/UART2_CTS: track 0.00 -> 32.7 mm
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- added copper zone on B.Cu, net GNDPWR
- removed copper zone on F.Cu, net GND
Other:
- board size 160 x 104.1 mm -> 170 x 100 mm

Commit message: Update: lots of refactoring and pin remap ..In chase for easier PCB routing PCB still not completed
Parts:
- removed C105: 100n, w_smd_capacitors:c_1206
- removed D503, D504: BAS85, w_smd_diode:sod80c
- removed IC503, IC504: PC817, w_pth_ic:dil_4-300
- removed Q404: BC847, SMD_Packages:SOT23
- removed R709, R710: 33, w_smd_resistors:r_0805
- removed U103: 74AC14, w_smd_dil:so-14
- added C110: 100n, w_smd_capacitors:c_0805, F.Cu at (127.4, 83.7)
- added C111: 100n, w_smd_capacitors:c_0805, F.Cu at (93.6, 96.5)
- added C112: 100n, w_smd_capacitors:c_0805, F.Cu at (96.8, 82.9)
- added C113: 100n, w_smd_capacitors:c_0805, F.Cu at (93.9, 98.9)
- added C114: 100n, w_smd_capacitors:c_0805, F.Cu at (96.8, 86.5)
- added C320: 100n, w_smd_capacitors:c_1206, B.Cu at (150.6, 61.0)
- added C503: 2.2u 6.3V Ta, w_smd_capacitors:c_tant_B, F.Cu at (140.5, 143.7)
- added C622: 1u MKT, w_pth_capacitors:cnp_7x6mm, F.Cu at (148.8, 159.3)
- added C623: 100n, w_smd_capacitors:c_1206, F.Cu at (127.9, 147.9)
- added D610: BAS85, w_smd_diode:sod80c, F.Cu at (147.3, 144.9)
- added D611: BAS85, w_smd_diode:sod80c, F.Cu at (135.5, 147.4)
- added Q501: BC847, SMD_Packages:SOT23, F.Cu at (140.5, 143.7)
- added R513: 3.3k, w_smd_resistors:r_1206, F.Cu at (140.5, 143.7)
- added R514, R515: 10k, w_smd_resistors:r_1206, F.Cu at (140.5, 143.7)
- added R615: 3.3k, w_smd_resistors:r_1206, F.Cu at (152.7, 150.5)
- added R616: Rt, w_smd_resistors:r_1210, F.Cu at (134.3, 141.9)
- added R617: 3.3k, w_smd_resistors:r_1206, F.Cu at (137.0, 152.9)
- added R618: 3.3k, w_smd_resistors:r_1206, F.Cu at (159.1, 144.5)
- added R705: 3.3k, w_smd_resistors:r_1206, F.Cu at (143.0, 77.2)
- C106, C107, C108, C109, C701, C707, D102, D701, R101: moved to B.Cu
- C618, C619: value 1u MKT -> 1.5u MKT
- C702, C703: footprint w_smd_capacitors:c_1206 -> w_smd_capacitors:c_0603
- C710, R715: moved to F.Cu
- C716: footprint w_smd_capacitors:c_0805 -> w_smd_capacitors:c_0603; moved to F.Cu
- P603: value LORAN In -> QUAD In; footprint w_conn_kk100:kk100_22-23-2021 -> w_conn_kk100:kk100_22-23-2041
- P604: value RSVD In -> LORAN In
- R104, R105: value 10 -> 200
- R505: value 4.7k -> 10k
- R507: value 4.7k -> 100
- R508: value 10k -> 3.3k
- R511, R512: value 200 -> 3.3k
- R704, R706, R707, R708, R719: footprint w_smd_resistors:r_1206 -> w_smd_resistors:r_0805
- moved C703 138.2 mm to (125.3, 92.8), turned to 270 degrees
- moved C705 135.1 mm to (119.5, 93.2)
- moved R713 134.9 mm to (123.5, 95.0), turned to 90 degrees
- moved C704 130.4 mm to (119.5, 96.7)
- moved C702 130.1 mm to (126.6, 92.8), turned to 270 degrees
- moved C106 126.1 mm to (84.9, 68.3), turned to 270 degrees
- moved C602 121.7 mm to (268.4, 128.0)
- moved C601 121.7 mm to (263.4, 128.0)
- moved C609 121.7 mm to (258.9, 141.3)
- moved C611 121.7 mm to (255.6, 141.3)
- moved C612 121.7 mm to (276.6, 133.6)
- moved P601 121.7 mm to (260.7, 151.0)
- moved P602 121.7 mm to (271.1, 151.0)
- moved R605 121.7 mm to (260.7, 146.3)
- moved R606 121.7 mm to (271.1, 146.3)
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Connections:
- net /CB_PO1 renamed /CB_PPS_OUT
- C618 pad 2: /uC STM32F407/ADC1_IN -> /uC STM32F407/ADC2_IN
- C619 pad 2: /uC STM32F407/ADC2_IN -> /uC STM32F407/ADC1_IN
- D606 pad 1: /uC STM32F407/ADC1_IN -> /uC STM32F407/ADC2_IN
- D607 pad 2: /uC STM32F407/ADC1_IN -> /uC STM32F407/ADC2_IN
- D608 pad 1: /uC STM32F407/ADC2_IN -> /uC STM32F407/ADC1_IN
- D609 pad 2: /uC STM32F407/ADC2_IN -> /uC STM32F407/ADC1_IN
- P103 pad 7: /CB_PO2 -> /CB_PPS_IN
- P103 pad 9: /CB_PPS -> (no net)
- P503 pad 1: Net-(D503-Pad2) -> GND
- P503 pad 2: Net-(D503-Pad1) -> Net-(P503-Pad2)
- P504 pad 1: Net-(D504-Pad2) -> GND
- P604 pad 1: Net-(C619-Pad1) -> Net-(C622-Pad1)
- Q403 pad 3: Net-(Q403-Pad3) -> /Relay optoisolation/RELAY3
- R104 pad 1: Net-(R104-Pad1) -> VDD
- R104 pad 2: /CB_PO2 -> /CB_PPS_IN
- R105 pad 1: Net-(R105-Pad1) -> /CB_PPS_IN
- R105 pad 2: /CB_PPS -> GND
- R107 pad 1: GND -> /CB_OSC
- R107 pad 2: /CB_OSC -> GND
- R505 pad 1: /Relay optoisolation/RELAY3 -> Net-(Q403-Pad1)
- R505 pad 2: Net-(Q403-Pad1) -> Net-(P503-Pad2)
- R507 pad 1: /Relay optoisolation/RELAY4 -> VDD
- R507 pad 2: Net-(Q404-Pad1) -> Net-(C502-Pad1)
- R508 pad 1: Net-(Q404-Pad1) -> VDD
- R508 pad 2: GND -> /Relay optoisolation/RELAY3
- R511 pad 1: Net-(IC503-Pad2) -> VDD
- R511 pad 2: Net-(Q403-Pad3) -> /Relay optoisolation/RELAY4
- R512 pad 1: Net-(IC504-Pad2) -> Net-(P503-Pad2)
- R512 pad 2: Net-(Q404-Pad3) -> Net-(C502-Pad1)
- R611 pad 2: /uC STM32F407/ADC1_IN -> /uC STM32F407/ADC2_IN
- R612 pad 1: /uC STM32F407/ADC1_IN -> /uC STM32F407/ADC2_IN
- R613 pad 2: /uC STM32F407/ADC2_IN -> /uC STM32F407/ADC1_IN
- R614 pad 1: /uC STM32F407/ADC2_IN -> /uC STM32F407/ADC1_IN
- U102 pad 1: /uC STM32F407/PROG_OUT1 -> /uC STM32F407/PPS3
- U102 pad 10: Net-(R104-Pad1) -> (no net)
- U102 pad 11: /uC STM32F407/PROG_OUT2 -> (no net)
- U102 pad 13: /uC STM32F407/PROG_OUT1 -> /uC STM32F407/PPS3
- U102 pad 3: /uC STM32F407/PROG_OUT2 -> /CB_PPS_IN
- U102 pad 4: Net-(R104-Pad1) -> /uC STM32F407/PPS_IN
- U102 pad 5: /uC STM32F407/PPS3 -> /CB_OSC
- U102 pad 6: Net-(R105-Pad1) -> Net-(R102-Pad2)
- U102 pad 8: Net-(R105-Pad1) -> (no net)
- U102 pad 9: /uC STM32F407/PPS3 -> (no net)
- U701 pad 15: (no net) -> /uC STM32F407/ADC3_IN
- U701 pad 63: /uC STM32F407/PPS1 -> (no net)
- U701 pad 64: /uC STM32F407/PPS2 -> (no net)
- U701 pad 65: /uC STM32F407/PPS3 -> /uC STM32F407/PPS2
- U701 pad 66: (no net) -> /uC STM32F407/PPS1
- U701 pad 93: (no net) -> /uC STM32F407/PPS3
- U701 pad 95: Net-(R709-Pad2) -> /uC STM32F407/PPS_IN
- U701 pad 96: Net-(R710-Pad2) -> (no net)
Routing:
- net /SPI interface/SPI_MISO: track 72.5 -> 19.4 mm
- net /Relay optoisolation/RELAY1: track 48.4 -> 0.00 mm
- net /CB_OSC: track 0.00 -> 45.1 mm, vias 0 -> 1
- net /SPI interface/SPI_SCK: track 87.8 -> 43.5 mm
- net VDD: track 147.2 -> 189.0 mm, vias 6 -> 4
- net /SPI interface/SPI_MOSI: track 53.6 -> 12.6 mm
- net /Relay optoisolation/RELAY2: track 40.2 -> 0.00 mm
- net /RS232 interface/UART2_RX: track 38.6 -> 0.00 mm
- net /SPI interface/SPI_STRB: track 85.2 -> 46.6 mm
- net /RS232 interface/UART2_TX: track 36.5 -> 0.00 mm
- net /Ethernet PHY/RMII_TX1: track 34.9 -> 0.00 mm
- net /RS232 interface/UART2_RTS: track 34.8 -> 0.00 mm
- net /uC STM32F407/OSC_IN: track 2.62 -> 35.5 mm, vias 0 -> 2
- net /Ethernet PHY/RMII_TX0: track 31.5 -> 0.00 mm
- net AGND: track 216.0 -> 246.0 mm, vias 3 -> 8
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- added copper zone on B.Cu, net AGND
- added copper zone on F.Cu, net VDD
