File: hardware/proc_board/loran_c_ethernet.sch (KiCad schematic (older format))
At the start: 41 parts, among them J201 RJ45, U201 LAN8720, X201 25MHz

Commit message: Update: fixed AGND zone on PCB
Parts:
- removed D201: LED_ETH, symbol LED_X2
- added D201: LED_ETH, symbol LED_x2
- C201, C203: footprint w_smd_capacitors:c_1206 -> w_smd_resistors:r_0805
- C205: footprint w_smd_capacitors:c_0603 -> w_smd_resistors:r_0805
- J201: footprint (none) -> Connect:RJ45_8
- R203, R204, R205: footprint w_smd_resistors:r_1206 -> w_smd_resistors:r_0805
- TR201: footprint (none) -> ts8121:TS8121
- X201: footprint (none) -> w_crystal:crystal_hc-49u
Changed lines of the file:
@@
 F 0 "J201" H 9750 3550 60  0000 C CNN
 F 1 "RJ45" H 9400 3550 60  0000 C CNN
-F 2 "" H 9550 3050 60  0001 C CNN
+F 2 "Connect:RJ45_8" H 9550 3050 60  0001 C CNN
 F 3 "" H 9550 3050 60  0000 C CNN
 	1    9550 3050
@@
 F 0 "TR201" H 7500 3450 50  0000 C CNN
 F 1 "TS8121" H 7500 2125 50  0000 C CNN
-F 2 "" H 7125 3150 60  0001 C CNN
+F 2 "ts8121:TS8121" H 7125 3150 60  0001 C CNN
 F 3 "" H 7125 3150 60  0000 C CNN
 	1    7500 2850
@@
 F 0 "X201" H 2800 4800 60  0000 C CNN
 F 1 "25MHz" H 2800 4500 60  0000 C CNN
-F 2 "" H 2800 4650 60  0001 C CNN
+F 2 "w_crystal:crystal_hc-49u" H 2800 4650 60  0001 C CNN
 F 3 "" H 2800 4650 60  0000 C CNN
 	1    2800 4650
@@
 F 0 "C203" H 3100 5250 40  0000 L CNN
 F 1 "22p" H 3106 5065 40  0000 L CNN
-F 2 "w_smd_capacitors:c_1206" H 3138 5000 30  0001 C CNN
+F 2 "w_smd_resistors:r_0805" H 3138 5000 30  0001 C CNN
 F 3 "" H 3100 5150 60  0000 C CNN
 	1    3100 5150
@@
 F 0 "C201" H 2500 5250 40  0000 L CNN
 F 1 "22p" H 2506 5065 40  0000 L CNN
-F 2 "w_smd_capacitors:c_1206" H 2538 5000 30  0001 C CNN
+F 2 "w_smd_resistors:r_0805" H 2538 5000 30  0001 C CNN
 F 3 "" H 2500 5150 60  0000 C CNN
 	1    2500 5150
@@
 F 0 "C205" H 3700 5350 40  0000 L CNN
 F 1 "470p" H 3706 5165 40  0000 L CNN
-F 2 "w_smd_capacitors:c_0603" H 3738 5100 30  0001 C CNN
+F 2 "w_smd_resistors:r_0805" H 3738 5100 30  0001 C CNN
 F 3 "" H 3700 5250 60  0000 C CNN
 	1    3700 5250
@@
 F 0 "R205" V 2950 3850 40  0000 C CNN
 F 1 "33" V 2907 4051 40  0000 C CNN
-F 2 "w_smd_resistors:r_1206" V 2830 4050 30  0001 C CNN
+F 2 "w_smd_resistors:r_0805" V 2830 4050 30  0001 C CNN
 F 3 "" H 2900 4050 30  0000 C CNN
 	1    2900 4050
@@
 F 0 "R203" V 2950 3300 40  0000 C CNN
 F 1 "33" V 2907 3501 40  0000 C CNN
-F 2 "w_smd_resistors:r_1206" V 2830 3500 30  0001 C CNN
+F 2 "w_smd_resistors:r_0805" V 2830 3500 30  0001 C CNN
 F 3 "" H 2900 3500 30  0000 C CNN
 	1    2900 3500
@@
 F 0 "R204" V 2950 3450 40  0000 C CNN
 F 1 "33" V 2907 3651 40  0000 C CNN
-F 2 "w_smd_resistors:r_1206" V 2830 3650 30  0001 C CNN
+F 2 "w_smd_resistors:r_0805" V 2830 3650 30  0001 C CNN
 F 3 "" H 2900 3650 30  0000 C CNN
 	1    2900 3650
@@
 Wire Wire Line
 	5850 4800 5850 5000
-$Comp
-L LED_X2 D201
-U 1 1 52EED8E3
-P 7250 4600
-F 0 "D201" H 7250 4750 50  0000 C CNN
-F 1 "LED_ETH" H 7250 4250 50  0000 C CNN
-F 2 "" H 7250 4600 60  0000 C CNN
-F 3 "" H 7250 4600 60  0000 C CNN
-	1    7250 4600
-	0    1    1    0
-$EndComp
 Wire Wire Line
 	7050 4200 7050 4250
@@
 Text Notes 2500 2100 0    39   ~ 0
 Place C204 close to pin 9 of U201
+$Comp
+L LED_x2 D201
+U 1 1 530E562A
+P 7250 4600
+F 0 "D201" H 7250 4750 50  0000 C CNN
+F 1 "LED_ETH" H 7250 4250 50  0000 C CNN
+F 2 "" H 7250 4600 60  0000 C CNN
+F 3 "" H 7250 4600 60  0000 C CNN
+	1    7250 4600
+	0    1    1    0
+$EndComp
 $EndSCHEMATC
