File: hardware/proc_board/loran_c_interfacing.sch (KiCad schematic (older format))
At the start: 18 parts, among them P401 SPI Bus A, P402 SPI Bus B, U401 74AC14, U402 74AC14

Commit message: Update: fixed AGND zone on PCB
Parts:
- U401, U402: footprint w_smd_dil:so-16 -> w_smd_dil:so-14
Changed lines of the file:
@@
 F 0 "U401" H 5750 1800 40  0000 C CNN
 F 1 "74AC14" H 5800 1600 40  0000 C CNN
-F 2 "w_smd_dil:so-16" H 5600 1700 60  0001 C CNN
+F 2 "w_smd_dil:so-14" H 5600 1700 60  0001 C CNN
 F 3 "" H 5600 1700 60  0000 C CNN
 	1    5600 1700
@@
 F 0 "U401" H 5750 2400 40  0000 C CNN
 F 1 "74AC14" H 5800 2200 40  0000 C CNN
-F 2 "w_smd_dil:so-16" H 5600 2300 60  0001 C CNN
+F 2 "w_smd_dil:so-14" H 5600 2300 60  0001 C CNN
 F 3 "" H 5600 2300 60  0000 C CNN
 	6    5600 2300
@@
 F 0 "U401" H 5750 2750 40  0000 C CNN
 F 1 "74AC14" H 5800 2550 40  0000 C CNN
-F 2 "w_smd_dil:so-16" H 5600 2650 60  0001 C CNN
+F 2 "w_smd_dil:so-14" H 5600 2650 60  0001 C CNN
 F 3 "" H 5600 2650 60  0000 C CNN
 	2    5600 2650
@@
 F 0 "U401" H 5750 3100 40  0000 C CNN
 F 1 "74AC14" H 5800 2900 40  0000 C CNN
-F 2 "w_smd_dil:so-16" H 5600 3000 60  0001 C CNN
+F 2 "w_smd_dil:so-14" H 5600 3000 60  0001 C CNN
 F 3 "" H 5600 3000 60  0000 C CNN
 	5    5600 3000
@@
 F 0 "U401" H 5750 3450 40  0000 C CNN
 F 1 "74AC14" H 5800 3250 40  0000 C CNN
-F 2 "w_smd_dil:so-16" H 5600 3350 60  0001 C CNN
+F 2 "w_smd_dil:so-14" H 5600 3350 60  0001 C CNN
 F 3 "" H 5600 3350 60  0000 C CNN
 	3    5600 3350
@@
 F 0 "U401" H 5750 3800 40  0000 C CNN
 F 1 "74AC14" H 5800 3600 40  0000 C CNN
-F 2 "w_smd_dil:so-16" H 5600 3700 60  0001 C CNN
+F 2 "w_smd_dil:so-14" H 5600 3700 60  0001 C CNN
 F 3 "" H 5600 3700 60  0000 C CNN
 	4    5600 3700
@@
 F 0 "U402" H 5750 4400 40  0000 C CNN
 F 1 "74AC14" H 5800 4200 40  0000 C CNN
-F 2 "w_smd_dil:so-16" H 5600 4300 60  0001 C CNN
+F 2 "w_smd_dil:so-14" H 5600 4300 60  0001 C CNN
 F 3 "" H 5600 4300 60  0000 C CNN
 	1    5600 4300
@@
 F 0 "U402" H 5750 5000 40  0000 C CNN
 F 1 "74AC14" H 5800 4800 40  0000 C CNN
-F 2 "w_smd_dil:so-16" H 5600 4900 60  0001 C CNN
+F 2 "w_smd_dil:so-14" H 5600 4900 60  0001 C CNN
 F 3 "" H 5600 4900 60  0000 C CNN
 	6    5600 4900
@@
 F 0 "U402" H 5750 5350 40  0000 C CNN
 F 1 "74AC14" H 5800 5150 40  0000 C CNN
-F 2 "w_smd_dil:so-16" H 5600 5250 60  0001 C CNN
+F 2 "w_smd_dil:so-14" H 5600 5250 60  0001 C CNN
 F 3 "" H 5600 5250 60  0000 C CNN
 	3    5600 5250
@@
 F 0 "U402" H 5750 5700 40  0000 C CNN
 F 1 "74AC14" H 5800 5500 40  0000 C CNN
-F 2 "w_smd_dil:so-16" H 5600 5600 60  0001 C CNN
+F 2 "w_smd_dil:so-14" H 5600 5600 60  0001 C CNN
 F 3 "" H 5600 5600 60  0000 C CNN
 	4    5600 5600
@@
 F 0 "U402" H 5750 6050 40  0000 C CNN
 F 1 "74AC14" H 5800 5850 40  0000 C CNN
-F 2 "w_smd_dil:so-16" H 5600 5950 60  0001 C CNN
+F 2 "w_smd_dil:so-14" H 5600 5950 60  0001 C CNN
 F 3 "" H 5600 5950 60  0000 C CNN
 	2    5600 5950
@@
 F 0 "U402" H 5750 6400 40  0000 C CNN
 F 1 "74AC14" H 5800 6200 40  0000 C CNN
-F 2 "w_smd_dil:so-16" H 5600 6300 60  0001 C CNN
+F 2 "w_smd_dil:so-14" H 5600 6300 60  0001 C CNN
 F 3 "" H 5600 6300 60  0000 C CNN
 	5    5600 6300
