File: hardware/proc_board/loran_c_relay.sch (KiCad schematic (older format))
At the start: 29 parts, among them IC501 PC817, IC502 PC817, P501 RELAY A, P502 RELAY B, P503 RELAY C, P504 RELAY D, Q501 BC847, Q502 BC847, Q503 BC847, Q504 BC847

Commit message: Update: fixed AGND zone on PCB
Parts:
- C502: footprint (none) -> w_smd_capacitors:c_1206
Changed lines of the file:
@@
 F 0 "C502" H 6350 6100 40  0000 L CNN
 F 1 "100n" H 6356 5915 40  0000 L CNN
-F 2 "" H 6388 5850 30  0000 C CNN
+F 2 "w_smd_capacitors:c_1206" H 6388 5850 30  0001 C CNN
 F 3 "" H 6350 6000 60  0000 C CNN
 	1    6350 6000
