File: hardware/proc_board/loran_c_rs232.sch (KiCad schematic (older format))
At the start: 28 parts, among them P301 UART1 3V3, P302 DB9 Ribbon 2, P303 DB9 Ribbon 1, P304 UART_SEL, U301 ST3232, U302 ST3232, U303 ST3232

Commit message: Update: fixed AGND zone on PCB
Parts:
- P304: footprint (none) -> Pin_Headers:Pin_Header_Straight_1x02
Changed lines of the file:
@@
 F 0 "P304" V 2750 8150 40  0000 C CNN
 F 1 "UART_SEL" V 2650 8150 40  0000 C CNN
-F 2 "" H 2700 8150 60  0000 C CNN
+F 2 "Pin_Headers:Pin_Header_Straight_1x02" H 2700 8150 60  0001 C CNN
 F 3 "" H 2700 8150 60  0000 C CNN
 	1    2700 8150
