File: hardware/proc_board/loran_c_uc.sch (KiCad schematic (older format))
At the start: 36 parts, among them U701 STM32F407VG, X701 32.768KHz

Commit message: Update: fixed AGND zone on PCB
Parts:
- C706, C707, C708, C709, C710, C716: footprint w_smd_capacitors:c_1206 -> w_smd_capacitors:c_0805
- R703, R704, R706, R707, R708, R713, R715: footprint w_smd_resistors:r_1206 -> w_smd_resistors:r_0805
- X701: footprint (none) -> w_crystal:crystal_tc-38_horiz
Changed lines of the file:
@@
 F 0 "C706" H 7600 1500 40  0000 L CNN
 F 1 "100n" H 7606 1315 40  0000 L CNN
-F 2 "w_smd_capacitors:c_1206" H 7638 1250 30  0001 C CNN
+F 2 "w_smd_capacitors:c_0805" H 7638 1250 30  0001 C CNN
 F 3 "" H 7600 1400 60  0000 C CNN
 	1    7600 1400
@@
 F 0 "C707" H 7900 1500 40  0000 L CNN
 F 1 "100n" H 7906 1315 40  0000 L CNN
-F 2 "w_smd_capacitors:c_1206" H 7938 1250 30  0001 C CNN
+F 2 "w_smd_capacitors:c_0805" H 7938 1250 30  0001 C CNN
 F 3 "" H 7900 1400 60  0000 C CNN
 	1    7900 1400
@@
 F 0 "C708" H 8200 1500 40  0000 L CNN
 F 1 "100n" H 8206 1315 40  0000 L CNN
-F 2 "w_smd_capacitors:c_1206" H 8238 1250 30  0001 C CNN
+F 2 "w_smd_capacitors:c_0805" H 8238 1250 30  0001 C CNN
 F 3 "" H 8200 1400 60  0000 C CNN
 	1    8200 1400
@@
 F 0 "C709" H 8500 1500 40  0000 L CNN
 F 1 "100n" H 8506 1315 40  0000 L CNN
-F 2 "w_smd_capacitors:c_1206" H 8538 1250 30  0001 C CNN
+F 2 "w_smd_capacitors:c_0805" H 8538 1250 30  0001 C CNN
 F 3 "" H 8500 1400 60  0000 C CNN
 	1    8500 1400
@@
 F 0 "C710" H 8800 1500 40  0000 L CNN
 F 1 "100n" H 8806 1315 40  0000 L CNN
-F 2 "w_smd_capacitors:c_1206" H 8838 1250 30  0001 C CNN
+F 2 "w_smd_capacitors:c_0805" H 8838 1250 30  0001 C CNN
 F 3 "" H 8800 1400 60  0000 C CNN
 	1    8800 1400
@@
 F 0 "R713" V 6180 1450 40  0000 C CNN
 F 1 "100" V 6107 1451 40  0000 C CNN
-F 2 "w_smd_resistors:r_1206" V 6030 1450 30  0001 C CNN
+F 2 "w_smd_resistors:r_0805" V 6030 1450 30  0001 C CNN
 F 3 "" H 6100 1450 30  0000 C CNN
 	1    6100 1450
@@
 F 0 "R704" V 2130 1750 40  0000 C CNN
 F 1 "3.3k" V 2057 1751 40  0000 C CNN
-F 2 "w_smd_resistors:r_1206" V 1980 1750 30  0001 C CNN
+F 2 "w_smd_resistors:r_0805" V 1980 1750 30  0001 C CNN
 F 3 "" H 2050 1750 30  0000 C CNN
 	1    2050 1750
@@
 F 0 "R703" V 2080 6350 40  0000 C CNN
 F 1 "3.3k" V 2007 6351 40  0000 C CNN
-F 2 "w_smd_resistors:r_1206" V 1930 6350 30  0001 C CNN
+F 2 "w_smd_resistors:r_0805" V 1930 6350 30  0001 C CNN
 F 3 "" H 2000 6350 30  0000 C CNN
 	1    2000 6350
@@
 F 0 "R706" V 2700 7200 40  0000 C CNN
 F 1 "33" V 2657 7401 40  0000 C CNN
-F 2 "w_smd_resistors:r_1206" V 2580 7400 30  0001 C CNN
+F 2 "w_smd_resistors:r_0805" V 2580 7400 30  0001 C CNN
 F 3 "" H 2650 7400 30  0000 C CNN
 	1    2650 7400
@@
 F 0 "R707" V 2700 7300 40  0000 C CNN
 F 1 "33" V 2657 7501 40  0000 C CNN
-F 2 "w_smd_resistors:r_1206" V 2580 7500 30  0001 C CNN
+F 2 "w_smd_resistors:r_0805" V 2580 7500 30  0001 C CNN
 F 3 "" H 2650 7500 30  0000 C CNN
 	1    2650 7500
@@
 F 0 "R708" V 2700 7400 40  0000 C CNN
 F 1 "33" V 2657 7601 40  0000 C CNN
-F 2 "w_smd_resistors:r_1206" V 2580 7600 30  0001 C CNN
+F 2 "w_smd_resistors:r_0805" V 2580 7600 30  0001 C CNN
 F 3 "" H 2650 7600 30  0000 C CNN
 	1    2650 7600
@@
 F 0 "R715" V 2200 4000 40  0000 C CNN
 F 1 "33" V 2157 4201 40  0000 C CNN
-F 2 "w_smd_resistors:r_1206" V 2080 4200 30  0001 C CNN
+F 2 "w_smd_resistors:r_0805" V 2080 4200 30  0001 C CNN
 F 3 "" H 2150 4200 30  0000 C CNN
 	1    2150 4200
@@
 F 0 "C716" H 9100 1500 40  0000 L CNN
 F 1 "100n" H 9106 1315 40  0000 L CNN
-F 2 "w_smd_capacitors:c_1206" H 9138 1250 30  0001 C CNN
+F 2 "w_smd_capacitors:c_0805" H 9138 1250 30  0001 C CNN
 F 3 "" H 9100 1400 60  0000 C CNN
 	1    9100 1400
@@
 F 0 "X701" H 14850 8300 60  0000 C CNN
 F 1 "32.768KHz" H 14850 8200 60  0000 C CNN
-F 2 "" H 14850 8000 60  0000 C CNN
+F 2 "w_crystal:crystal_tc-38_horiz" H 14850 8000 60  0001 C CNN
 F 3 "" H 14850 8000 60  0000 C CNN
 	1    14850 8000
